Commit message: controller launch file made

File: src/practice_robotarm_description/urdf/practice_robotarm_gazebo.xacro (robot description, xacro)
@@ -4,10 +4,10 @@
         <xacro:if value="$(arg is_ignition)">
             <plugin filename="ign_ros2_control-system" name="ign_ros2_control::IgnitionROS2ControlPlugin">
-            <parameters>$(find practice_robotarm_controller)/config/practice_robotarm_controllers.yaml</parameters>
+                <parameters>$(find practice_robotarm_controller)/config/practice_robotarm_controllers.yaml</parameters>
             </plugin>
         </xacro:if>
         <xacro:unless value="$(arg is_ignition)">
             <plugin filename="gz_ros2_control-system" name="gz_ros2_control::GazeboSimROS2ControlPlugin">
-            <parameters>$(find practice_robotarm_controller)/config/practice_robotarm_controllers.yaml</parameters>
+                <parameters>$(find practice_robotarm_controller)/config/practice_robotarm_controllers.yaml</parameters>
             </plugin>
         </xacro:unless>

File: src/practice_robotarm_description/urdf/practice_robotarm_ros2_control.xacro (robot description, xacro)
@@ -1,6 +1,8 @@
 <?xml version="1.0"?>
 <robot xmlns:xacro="http://www.ros.org/wiki/xacro" name="practice_robotarm">
-    <xacro:property name="PI" value="3.14159"/>
-    <ros2_control type="system" name="RobotSystem">
+    <ros2_control name="RobotSystem" type="system">
+        <xacro:property name="PI" value="3.14159265359" />
+        <!-- ros2_control Gazebo -->
+        <!-- ROS 2 Humble -->
         <xacro:if value="$(arg is_ignition)">
             <hardware>
@@ -8,4 +10,5 @@
             </hardware>
         </xacro:if>
+        <!-- ROS 2 Iron or above -->
         <xacro:unless value="$(arg is_ignition)">
             <hardware>
@@ -15,6 +18,6 @@
         <joint name="joint_1">
             <command_interface name="position">
-                <param name="min">-${PI/2}</param>
-                <param name="max">${PI/2}</param>
+            <param name="min">-${PI / 2}</param>
+            <param name="max">${PI / 2}</param>
             </command_interface>
             <state_interface name="position"/>
@@ -22,6 +25,6 @@
         <joint name="joint_2">
             <command_interface name="position">
-                <param name="min">-${PI/2}</param>
-                <param name="max">${PI/2}</param>
+            <param name="min">-${PI / 2}</param>
+            <param name="max">${PI / 2}</param>
             </command_interface>
             <state_interface name="position"/>
@@ -29,6 +32,6 @@
         <joint name="joint_3">
             <command_interface name="position">
-                <param name="min">-${PI/2}</param>
-                <param name="max">${PI/2}</param>
+            <param name="min">-${PI / 2}</param>
+            <param name="max">${PI / 2}</param>
             </command_interface>
             <state_interface name="position"/>
@@ -36,6 +39,6 @@
         <joint name="joint_4">
             <command_interface name="position">
-                <param name="min">-${PI/2}</param>
-                <param name="max">0.0</param>
+            <param name="min">-${PI / 2}</param>
+            <param name="max">0.0</param>
             </command_interface>
             <state_interface name="position"/>
@@ -43,5 +46,5 @@
         <joint name="joint_5">
             <param name="mimic">joint_4</param>
-            <param name="multiplier">-1.0</param>
+            <param name="multiplier">-1</param>
         </joint>
     </ros2_control>
